File: 68_vag_PNP.kicad_pcb (KiCad board)
At the start: 2 copper layers, 154 x 159 mm, 173 parts, among them J1 Conn_01x01, J10 Conn_02x11_Odd_Even, J11 Conn_02x11_Odd_Even, J12 Conn_02x11_Odd_Even, J13 Conn_02x11_Odd_Even, J14 Conn_02x11_Odd_Even, J15 Conn_02x11_Odd_Even, J16 Conn_02x11_Odd_Even, J17 Conn_02x11_Odd_Even, J18 Conn_02x11_Odd_Even, J19 Conn_02x11_Odd_Even, J2 Conn_01x01, J20 Conn_02x11_Odd_Even, J21 Conn_02x11_Odd_Even, J22 Conn_02x11_Odd_Even, J23 Conn_02x11_Odd_Even, J24 Conn_01x01, J25 Conn_01x01, J26 Conn_01x01, J27 Conn_01x01, J28 Conn_01x01, J29 Conn_01x01, J3 Conn_01x01, J30 Conn_01x01, J31 Conn_01x01, J32 Conn_01x01, J33 Conn_01x01, J34 Conn_01x01, J35 Conn_01x01, J36 Conn_01x01, J37 Conn_01x01, J38 Conn_01x01, J39 Conn_01x01, J4 Conn_01x05, J40 Conn_01x01, J5 Conn_01x01, J6 Conn_01x05, J7 Conn_01x05, J8 Conn_01x05, J9 Conn_02x11_Odd_Even, P1 1123038-2, U1 VNLD5090, U2 VNLD5090, U3 molex_48pin_MRE, U4 ITEAD_HC-05

Commit message: draft
Parts:
- moved BT1 261.9 mm to (418.5, 128.9)
- moved C1 261.9 mm to (306.8, 73.2)
- moved C2 261.9 mm to (306.8, 76.3)
- moved C3 261.9 mm to (306.8, 86.4)
- moved C4 261.9 mm to (306.8, 89.7)
- moved C5 261.9 mm to (307.4, 128.6)
- moved D16 261.9 mm to (315.0, 61.7)
- moved D2 261.9 mm to (309.1, 77.3)
- moved D20 261.9 mm to (318.9, 61.7)
- moved D21 261.9 mm to (323.3, 57.8)
- moved D22 261.9 mm to (323.3, 61.7)
- moved D27 261.9 mm to (335.4, 57.7)
- moved D28 261.9 mm to (335.4, 61.7)
- moved D30 261.9 mm to (377.6, 48.9)
- moved D5 261.9 mm to (309.1, 84.1)
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Other:
- board size 154 x 159 mm -> 149 x 85 mm

Commit message: draft
Parts:
- moved U3 52.5 mm to (75.0, 45.0), turned to 0 degrees
Routing:
- net GND: vias 123 -> 122
- net (no net): vias 1 -> 2
Other:
- board size 149 x 85 mm -> 149 x 140 mm

Commit message: draft
Other:
- outline, holes or cut-outs redrawn
- board text added: "A1"
- board text added: "A2"
- board text added: "B1"
- board text added: "B2"
- board text added: "C1"
- board text added: "C2"
Changed lines of the file:
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@@
   (general
     (thickness 1.6)
-    (drawings 212)
+    (drawings 226)
     (tracks 1861)
     (zones 0)
@@
     (39 F.Mask user hide)
     (40 Dwgs.User user)
-    (41 Cmts.User user hide)
+    (41 Cmts.User user)
     (42 Eco1.User user)
     (43 Eco2.User user)
@@
     )
   )
+  (gr_text C1 (at 45.5 148.5) (layer Dwgs.User)
+    (effects (font (size 10 10) (thickness 0.15)))
+  )
+  (dimension 7.725108 (width 0.15) (layer Dwgs.User)
+    (gr_text "7.725 mm" (at 40.3 147.955 90) (layer Dwgs.User)
+      (effects (font (size 1 1) (thickness 0.15)))
+    )
+    (feature1 (pts (xy 31.75 144.092446) (xy 39.586421 144.092446)))
+    (feature2 (pts (xy 31.75 151.817554) (xy 39.586421 151.817554)))
+    (crossbar (pts (xy 39 151.817554) (xy 39 144.092446)))
+    (arrow1a (pts (xy 39 144.092446) (xy 39.586421 145.21895)))
+    (arrow1b (pts (xy 39 144.092446) (xy 38.413579 145.21895)))
+    (arrow2a (pts (xy 39 151.817554) (xy 39.586421 150.69105)))
+    (arrow2b (pts (xy 39 151.817554) (xy 38.413579 150.69105)))
+  )
+  (gr_text C2 (at 148 61.5) (layer Dwgs.User)
+    (effects (font (size 10 10) (thickness 0.15)))
+  )
+  (gr_text B2 (at 206 34) (layer Dwgs.User)
+    (effects (font (size 10 10) (thickness 0.15)))
+  )
+  (gr_text A2 (at 78 -13.5) (layer Dwgs.User)
+    (effects (font (size 10 10) (thickness 0.15)))
+  )
+  (gr_text A1 (at 23.5 173.5) (layer Dwgs.User)
+    (effects (font (size 10 10) (thickness 0.15)))
+  )
+  (gr_text B1 (at -6 84) (layer Dwgs.User)
+    (effects (font (size 10 10) (thickness 0.15)))
+  )
+  (dimension 124 (width 0.15) (layer Dwgs.User)
+    (gr_text "124.000 mm" (at 4.7 82 90) (layer Dwgs.User)
+      (effects (font (size 1 1) (thickness 0.15)))
+    )
+    (feature1 (pts (xy 31.5 20) (xy 5.413579 20)))
+    (feature2 (pts (xy 31.5 144) (xy 5.413579 144)))
+    (crossbar (pts (xy 6 144) (xy 6 20)))
+    (arrow1a (pts (xy 6 20) (xy 6.586421 21.126504)))
+    (arrow1b (pts (xy 6 20) (xy 5.413579 21.126504)))
+    (arrow2a (pts (xy 6 144) (xy 6.586421 142.873496)))
+    (arrow2b (pts (xy 6 144) (xy 5.413579 142.873496)))
+  )
+  (dimension 8 (width 0.15) (layer Dwgs.User)
+    (gr_text "8.000 mm" (at 24 165.3) (layer Dwgs.User)
+      (effects (font (size 1 1) (thickness 0.15)))
+    )
+    (feature1 (pts (xy 20 148) (xy 20 164.586421)))
+    (feature2 (pts (xy 28 148) (xy 28 164.586421)))
+    (crossbar (pts (xy 28 164) (xy 20 164)))
+    (arrow1a (pts (xy 20 164) (xy 21.126504 163.413579)))
+    (arrow1b (pts (xy 20 164) (xy 21.126504 164.586421)))
+    (arrow2a (pts (xy 28 164) (xy 26.873496 163.413579)))
+    (arrow2b (pts (xy 28 164) (xy 26.873496 164.586421)))
+  )
+  (dimension 7.725108 (width 0.15) (layer Dwgs.User)
+    (gr_text "7.725 mm" (at 149.3 51.435 270) (layer Dwgs.User)
+      (effects (font (size 1 1) (thickness 0.15)))
+    )
+    (feature1 (pts (xy 140.97 55.297554) (xy 148.586421 55.297554)))
+    (feature2 (pts (xy 140.97 47.572446) (xy 148.586421 47.572446)))
+    (crossbar (pts (xy 148 47.572446) (xy 148 55.297554)))
+    (arrow1a (pts (xy 148 55.297554) (xy 147.413579 54.17105)))
+    (arrow1b (pts (xy 148 55.297554) (xy 148.586421 54.17105)))
+    (arrow2a (pts (xy 148 47.572446) (xy 147.413579 48.69895)))
+    (arrow2b (pts (xy 148 47.572446) (xy 148.586421 48.69895)))
+  )
+  (dimension 117 (width 0.15) (layer Dwgs.User)
+    (gr_text "117.000 mm" (at 78.5 -7.299999) (layer Dwgs.User)
+      (effects (font (size 1 1) (thickness 0.15)))
+    )
+    (feature1 (pts (xy 20 51.5) (xy 20 -6.58642)))
+    (feature2 (pts (xy 137 51.5) (xy 137 -6.58642)))
+    (crossbar (pts (xy 137 -5.999999) (xy 20 -5.999999)))
+    (arrow1a (pts (xy 20 -5.999999) (xy 21.126504 -6.58642)))
+    (arrow1b (pts (xy 20 -5.999999) (xy 21.126504 -5.413578)))
+    (arrow2a (pts (xy 137 -5.999999) (xy 135.873496 -6.58642)))
+    (arrow2b (pts (xy 137 -5.999999) (xy 135.873496 -5.413578)))
+  )
+  (dimension 27.5 (width 0.15) (layer Dwgs.User)
+    (gr_text "27.500 mm" (at 200.3 33.75 90) (layer Dwgs.User)
+      (effects (font (size 1 1) (thickness 0.15)))
+    )
+    (feature1 (pts (xy 141 20) (xy 199.586421 20)))
+    (feature2 (pts (xy 141 47.5) (xy 199.586421 47.5)))
+    (crossbar (pts (xy 199 47.5) (xy 199 20)))
+    (arrow1a (pts (xy 199 20) (xy 199.586421 21.126504)))
+    (arrow1b (pts (xy 199 20) (xy 198.413579 21.126504)))
+    (arrow2a (pts (xy 199 47.5) (xy 199.586421 46.373496)))
+    (arrow2b (pts (xy 199 47.5) (xy 198.413579 46.373496)))
+  )
+  (gr_circle (center 140.97 51.435) (end 144.78 52.07) (layer Edge.Cuts) (width 0.2))
+  (gr_circle (center 31.75 147.955) (end 35.56 148.59) (layer Edge.Cuts) (width 0.2))
   (dimension 140 (width 0.15) (layer Dwgs.User)
     (gr_text "140.000 mm" (at 183.596461 90 90) (layer Dwgs.User)
@@
   )
   (via (at 359.49 28.062) (size 0.6) (drill 0.3) (layers F.Cu B.Cu) (net 0))
+  (via (at 339.043 88.133) (size 0.6) (drill 0.3) (layers F.Cu B.Cu) (net 0))
   (segment (start 304.28 89.6824) (end 304.28 90.835) (width 1.0668) (layer F.Cu) (net 1))
   (segment (start 304.28 90.835) (end 304.88 91.435) (width 1.0668) (layer F.Cu) (net 1))
@@
   (via (at 325.962 62.86) (size 0.6) (drill 0.3) (layers F.Cu B.Cu) (net 1))
   (via (at 313.262 65.019) (size 0.6) (drill 0.3) (layers F.Cu B.Cu) (net 1))
-  (via (at 339.043 88.133) (size 0.6) (drill 0.3) (layers F.Cu B.Cu) (net 0))
   (via (at 341.456 115.565) (size 0.6) (drill 0.3) (layers F.Cu B.Cu) (net 1))
   (via (at 370.92 114.549) (size 0.6) (drill 0.3) (layers F.Cu B.Cu) (net 1))
