File: 68_vag_PNP.kicad_pcb (KiCad board)
At the start: 2 copper layers, 149 x 140 mm, 173 parts, among them J1 Conn_01x01, J10 Conn_02x11_Odd_Even, J11 Conn_02x11_Odd_Even, J12 Conn_02x11_Odd_Even, J13 Conn_02x11_Odd_Even, J14 Conn_02x11_Odd_Even, J15 Conn_02x11_Odd_Even, J16 Conn_02x11_Odd_Even, J17 Conn_02x11_Odd_Even, J18 Conn_02x11_Odd_Even, J19 Conn_02x11_Odd_Even, J2 Conn_01x01, J20 Conn_02x11_Odd_Even, J21 Conn_02x11_Odd_Even, J22 Conn_02x11_Odd_Even, J23 Conn_02x11_Odd_Even, J24 Conn_01x01, J25 Conn_01x01, J26 Conn_01x01, J27 Conn_01x01, J28 Conn_01x01, J29 Conn_01x01, J3 Conn_01x01, J30 Conn_01x01, J31 Conn_01x01, J32 Conn_01x01, J33 Conn_01x01, J34 Conn_01x01, J35 Conn_01x01, J36 Conn_01x01, J37 Conn_01x01, J38 Conn_01x01, J39 Conn_01x01, J4 Conn_01x05, J40 Conn_01x01, J5 Conn_01x01, J6 Conn_01x05, J7 Conn_01x05, J8 Conn_01x05, J9 Conn_02x11_Odd_Even, P1 1123038-2, U1 VNLD5090, U2 VNLD5090, U3 molex_48pin_MRE, U4 ITEAD_HC-05

Commit message: R0.1 draft, pre-auto-route
Parts:
- removed J1, J3: Conn_01x01, Connector_PinSocket_2.00mm:PinSocket_1x01_P2.00mm_Vertical
- removed J20, J21, J22, J23: Conn_02x11_Odd_Even, Connector_PinHeader_2.54mm:PinHeader_2x11_P2.54mm_Vertical
- removed W2A1, W2B1, W2C1, W2D1, W2E1, W2F1, W2G1, W2H1, W2I1, W2J1, W2K1, W2M1, W2N1, W2O1, W2P1, W2Q1, W2R1, W3A1, W3B1, W3C1, W3D1, W3E1, W3F1, W3H1, W3I1, W3J1, W3K1, W3L1, W3M1, W3N1, W3O1, W3P1, W3Q1, W3S1, W3T1, W3U1, W3V1, W3W1, W3X1, W3Y1, W3Z1, W4A1, W4AA1, W4AB1, W4AC1, W4AD1, W4AE1, W4AF1, W4AG1, W4AH1, W4B1, W4C1, W4D1, W4E1, W4F1, W4H1, W4I1, W4J1, W4K1, W4L1, W4M1, W4N1, W4O1, W4P1, W4R1, W4S1, W4T1, W4U1, W4V1, W4W1, W4X1, W4Z1: TestPoint_2Pole, rusEFI_Modules:SM0805_jumper
- added G1: Disclaimer, rusEFI_Modules:Off_Road_Disclaimer, F.Cu at (26.0, 114.3)
- added J10: Conn_01x01, Connector_PinHeader_2.54mm:PinHeader_1x01_P2.54mm_Vertical, B.Cu at (136.5, 115.6)
- added J11: Conn_01x01, Connector_PinHeader_2.54mm:PinHeader_1x01_P2.54mm_Vertical, B.Cu at (136.5, 118.1)
- added J14: Conn_01x01, Connector_PinHeader_2.54mm:PinHeader_1x01_P2.54mm_Vertical, B.Cu at (88.3, 75.6)
- added J16: Conn_01x01, Connector_PinHeader_2.54mm:PinHeader_1x01_P2.54mm_Vertical, B.Cu at (136.5, 120.7)
- added J18: Conn_01x01, Connector_PinHeader_2.54mm:PinHeader_1x01_P2.54mm_Vertical, B.Cu at (136.5, 123.2)
- added J201: Conn_01x05, Connector_PinSocket_2.54mm:PinSocket_1x05_P2.54mm_Vertical, B.Cu at (140.3, 109.9)
- added J202: Conn_01x05, Connector_PinSocket_2.54mm:PinSocket_1x05_P2.54mm_Vertical, B.Cu at (137.8, 109.9)
- added J41: Conn_01x01, TestPoint:TestPoint_Pad_4.0x4.0mm, B.Cu at (152.4, 63.5)
- added J42: Conn_01x01, Connector_PinHeader_2.54mm:PinHeader_1x01_P2.54mm_Vertical, F.Cu at (152.4, 63.5)
- added J45: Conn_01x01, Connector_PinHeader_2.54mm:PinHeader_1x01_P2.54mm_Vertical, F.Cu at (38.1, 109.2)
- added J46: Conn_01x01, Connector_PinHeader_2.54mm:PinHeader_1x01_P2.54mm_Vertical, F.Cu at (26.7, 101.0)
- added J47: Conn_01x01, Connector_PinHeader_2.54mm:PinHeader_1x01_P2.54mm_Vertical, F.Cu at (111.1, 48.9)
- added J48: Conn_01x01, Connector_PinHeader_2.54mm:PinHeader_1x01_P2.54mm_Vertical, F.Cu at (38.1, 83.8)
- added J49: Conn_01x01, Connector_PinHeader_2.54mm:PinHeader_1x01_P2.54mm_Vertical, F.Cu at (38.1, 78.7)
- added J52: Conn_01x01, Connector_PinHeader_2.54mm:PinHeader_1x01_P2.54mm_Vertical, F.Cu at (121.9, 48.9)
- added J53: Conn_01x01, Connector_PinHeader_2.54mm:PinHeader_1x01_P2.54mm_Vertical, F.Cu at (159.4, 48.9)
- added J56: Conn_01x01, Connector_PinHeader_2.54mm:PinHeader_1x01_P2.54mm_Vertical, F.Cu at (58.4, 48.3)
- added J57: Conn_01x01, Connector_PinHeader_2.54mm:PinHeader_1x01_P2.54mm_Vertical, F.Cu at (32.4, 97.8)
- added J58: Conn_01x01, Connector_PinHeader_2.54mm:PinHeader_1x01_P2.54mm_Vertical, F.Cu at (32.4, 92.7)
- added J6: Conn_01x01, Connector_PinHeader_2.54mm:PinHeader_1x01_P2.54mm_Vertical, B.Cu at (136.5, 125.7)
- added J62: Conn_01x01, Connector_PinHeader_2.54mm:PinHeader_1x01_P2.54mm_Vertical, F.Cu at (32.4, 87.6)
- added J63: Conn_01x01, Connector_PinHeader_2.54mm:PinHeader_1x01_P2.54mm_Vertical, F.Cu at (32.4, 82.5)
- added J64: Conn_01x01, Connector_PinHeader_2.54mm:PinHeader_1x01_P2.54mm_Vertical, F.Cu at (32.4, 90.2)
- added J65: Conn_01x01, Connector_PinHeader_2.54mm:PinHeader_1x01_P2.54mm_Vertical, F.Cu at (26.7, 92.7)
- added J67: Conn_01x01, Connector_PinHeader_2.54mm:PinHeader_1x01_P2.54mm_Vertical, F.Cu at (38.1, 76.2)
- added J68: Conn_01x01, Connector_PinHeader_2.54mm:PinHeader_1x01_P2.54mm_Vertical, F.Cu at (38.1, 73.7)
- added J69: Conn_01x01, Connector_PinHeader_2.54mm:PinHeader_1x01_P2.54mm_Vertical, F.Cu at (38.1, 99.1)
- added J70: Conn_01x01, Connector_PinHeader_2.54mm:PinHeader_1x01_P2.54mm_Vertical, F.Cu at (38.1, 96.5)
- added J71: Conn_01x01, Connector_PinHeader_2.54mm:PinHeader_1x01_P2.54mm_Vertical, F.Cu at (32.4, 100.3)
- added J72: Conn_01x01, Connector_PinHeader_2.54mm:PinHeader_1x01_P2.54mm_Vertical, F.Cu at (38.1, 101.6)
- added J9: Conn_01x01, Connector_PinHeader_2.54mm:PinHeader_1x01_P2.54mm_Vertical, B.Cu at (136.5, 113.0)
- added JA12: Conn_02x11_Odd_Even, Connector_PinHeader_2.54mm:PinHeader_2x11_P2.54mm_Vertical, F.Cu at (112.4, 134.0)
- added JA13: Conn_02x11_Odd_Even, Connector_PinHeader_2.54mm:PinHeader_2x11_P2.54mm_Vertical, F.Cu at (112.4, 139.1)
- added JA14: Conn_02x11_Odd_Even, Connector_PinHeader_2.54mm:PinHeader_2x11_P2.54mm_Vertical, F.Cu at (112.4, 144.1)
- added JA15: Conn_02x11_Odd_Even, Connector_PinHeader_2.54mm:PinHeader_2x11_P2.54mm_Vertical, F.Cu at (112.4, 149.2)
- added JA16: Conn_02x11_Odd_Even, Connector_PinHeader_2.54mm:PinHeader_2x11_P2.54mm_Vertical, F.Cu at (112.4, 154.3)
- added LOGO3: LOGO, Symbol:OSHW-Logo2_7.3x6mm_SilkScreen, F.Cu at (36.2, 121.3)
- added W1: TestPoint_2Pole, rusEFI_Modules:SM0805_jumper, F.Cu at (131.4, 38.7)
- added W10: TestPoint_2Pole, rusEFI_Modules:SM0805_jumper, F.Cu at (90.8, 38.7)
- added W11: TestPoint_2Pole, rusEFI_Modules:SM0805_jumper, F.Cu at (87.0, 44.5)
- added W12: TestPoint_2Pole, rusEFI_Modules:SM0805_jumper, F.Cu at (83.2, 38.7)
- added W13: TestPoint_2Pole, rusEFI_Modules:SM0805_jumper, F.Cu at (79.4, 44.5)
- added W14: TestPoint_2Pole, rusEFI_Modules:SM0805_jumper, F.Cu at (74.9, 38.7)
- added W15: TestPoint_2Pole, rusEFI_Modules:SM0805_jumper, F.Cu at (71.1, 44.5)
- added W16: TestPoint_2Pole, rusEFI_Modules:SM0805_jumper, F.Cu at (67.3, 38.7)
- added W17: TestPoint_2Pole, rusEFI_Modules:SM0805_jumper, F.Cu at (63.5, 44.5)
- added W18: TestPoint_2Pole, rusEFI_Modules:SM0805_jumper, F.Cu at (59.7, 38.7)
- added W19: TestPoint_2Pole, rusEFI_Modules:SM0805_jumper, F.Cu at (55.9, 44.5)
- added W2: TestPoint_2Pole, rusEFI_Modules:SM0805_jumper, F.Cu at (123.2, 38.7)
- added W20: TestPoint_2Pole, rusEFI_Modules:SM0805_jumper, F.Cu at (52.1, 38.7)
- added W21: TestPoint_2Pole, rusEFI_Modules:SM0805_jumper, F.Cu at (48.3, 44.5)
- added W22: TestPoint_2Pole, rusEFI_Modules:SM0805_jumper, F.Cu at (44.5, 38.7)
- added W23: TestPoint_2Pole, rusEFI_Modules:SM0805_jumper, F.Cu at (36.8, 38.7)
- added W24: TestPoint_2Pole, rusEFI_Modules:SM0805_jumper, F.Cu at (125.7, 38.7)
- added W25: TestPoint_2Pole, rusEFI_Modules:SM0805_jumper, F.Cu at (121.9, 44.5)
- added W26: TestPoint_2Pole, rusEFI_Modules:SM0805_jumper, F.Cu at (118.1, 38.7)
- added W27: TestPoint_2Pole, rusEFI_Modules:SM0805_jumper, F.Cu at (113.7, 44.5)
- added W28: TestPoint_2Pole, rusEFI_Modules:SM0805_jumper, F.Cu at (109.9, 38.7)
- added W29: TestPoint_2Pole, rusEFI_Modules:SM0805_jumper, F.Cu at (106.0, 44.5)
- added W3: TestPoint_2Pole, rusEFI_Modules:SM0805_jumper, F.Cu at (119.6, 44.5)
- added W30: TestPoint_2Pole, rusEFI_Modules:SM0805_jumper, F.Cu at (102.2, 38.7)
- added W31: TestPoint_2Pole, rusEFI_Modules:SM0805_jumper, F.Cu at (98.4, 44.5)
- added W32: TestPoint_2Pole, rusEFI_Modules:SM0805_jumper, F.Cu at (93.3, 38.7)
- added W33: TestPoint_2Pole, rusEFI_Modules:SM0805_jumper, F.Cu at (89.5, 44.5)
- added W34: TestPoint_2Pole, rusEFI_Modules:SM0805_jumper, F.Cu at (85.7, 38.7)
- added W35: TestPoint_2Pole, rusEFI_Modules:SM0805_jumper, F.Cu at (81.9, 44.5)
- added W36: TestPoint_2Pole, rusEFI_Modules:SM0805_jumper, F.Cu at (78.1, 38.7)
- added W37: TestPoint_2Pole, rusEFI_Modules:SM0805_jumper, F.Cu at (73.7, 44.5)
- added W38: TestPoint_2Pole, rusEFI_Modules:SM0805_jumper, F.Cu at (69.8, 38.7)
- added W39: TestPoint_2Pole, rusEFI_Modules:SM0805_jumper, F.Cu at (66.0, 44.5)
- added W4: TestPoint_2Pole, rusEFI_Modules:SM0805_jumper, F.Cu at (114.9, 38.7)
- added W40: TestPoint_2Pole, rusEFI_Modules:SM0805_jumper, F.Cu at (62.2, 38.7)
- added W41: TestPoint_2Pole, rusEFI_Modules:SM0805_jumper, F.Cu at (58.4, 44.5)
- added W42: TestPoint_2Pole, rusEFI_Modules:SM0805_jumper, F.Cu at (54.6, 38.7)
- added W43: TestPoint_2Pole, rusEFI_Modules:SM0805_jumper, F.Cu at (50.8, 44.5)
- added W44: TestPoint_2Pole, rusEFI_Modules:SM0805_jumper, F.Cu at (47.0, 38.7)
- added W45: TestPoint_2Pole, rusEFI_Modules:SM0805_jumper, F.Cu at (41.9, 38.7)
- added W46: TestPoint_2Pole, rusEFI_Modules:SM0805_jumper, F.Cu at (128.9, 44.5)
- added W47: TestPoint_2Pole, rusEFI_Modules:SM0805_jumper, F.Cu at (124.5, 44.5)
- added W48: TestPoint_2Pole, rusEFI_Modules:SM0805_jumper, F.Cu at (120.7, 38.7)
- added W49: TestPoint_2Pole, rusEFI_Modules:SM0805_jumper, F.Cu at (116.2, 44.5)
- added W5: TestPoint_2Pole, rusEFI_Modules:SM0805_jumper, F.Cu at (111.1, 44.5)
- added W50: TestPoint_2Pole, rusEFI_Modules:SM0805_jumper, F.Cu at (112.4, 38.7)
- added W51: TestPoint_2Pole, rusEFI_Modules:SM0805_jumper, F.Cu at (108.6, 44.5)
- added W52: TestPoint_2Pole, rusEFI_Modules:SM0805_jumper, F.Cu at (104.8, 38.7)
- added W53: TestPoint_2Pole, rusEFI_Modules:SM0805_jumper, F.Cu at (101.0, 44.5)
- added W54: TestPoint_2Pole, rusEFI_Modules:SM0805_jumper, F.Cu at (95.9, 38.7)
- added W55: TestPoint_2Pole, rusEFI_Modules:SM0805_jumper, F.Cu at (92.1, 44.5)
- added W56: TestPoint_2Pole, rusEFI_Modules:SM0805_jumper, F.Cu at (88.3, 38.7)
- added W57: TestPoint_2Pole, rusEFI_Modules:SM0805_jumper, F.Cu at (84.5, 44.5)
- added W58: TestPoint_2Pole, rusEFI_Modules:SM0805_jumper, F.Cu at (80.6, 38.7)
- added W59: TestPoint_2Pole, rusEFI_Modules:SM0805_jumper, F.Cu at (76.2, 44.5)
- added W6: TestPoint_2Pole, rusEFI_Modules:SM0805_jumper, F.Cu at (107.3, 38.7)
- added W60: TestPoint_2Pole, rusEFI_Modules:SM0805_jumper, F.Cu at (72.4, 38.7)
- added W61: TestPoint_2Pole, rusEFI_Modules:SM0805_jumper, F.Cu at (68.6, 44.5)
- added W62: TestPoint_2Pole, rusEFI_Modules:SM0805_jumper, F.Cu at (64.8, 38.7)
- added W63: TestPoint_2Pole, rusEFI_Modules:SM0805_jumper, F.Cu at (61.0, 44.5)
- added W64: TestPoint_2Pole, rusEFI_Modules:SM0805_jumper, F.Cu at (57.1, 38.7)
- added W65: TestPoint_2Pole, rusEFI_Modules:SM0805_jumper, F.Cu at (53.3, 44.5)
- added W66: TestPoint_2Pole, rusEFI_Modules:SM0805_jumper, F.Cu at (49.5, 38.7)
- added W67: TestPoint_2Pole, rusEFI_Modules:SM0805_jumper, F.Cu at (45.7, 44.5)
- added W68: TestPoint_2Pole, rusEFI_Modules:SM0805_jumper, F.Cu at (39.4, 38.7)
- added W7: TestPoint_2Pole, rusEFI_Modules:SM0805_jumper, F.Cu at (103.5, 44.5)
- added W8: TestPoint_2Pole, rusEFI_Modules:SM0805_jumper, F.Cu at (99.7, 38.7)
- added W9: TestPoint_2Pole, rusEFI_Modules:SM0805_jumper, F.Cu at (94.6, 44.5)
- J2: footprint Connector_PinSocket_2.00mm:PinSocket_1x01_P2.00mm_Vertical -> Connector_PinHeader_2.54mm:PinHeader_1x01_P2.54mm_Vertical
- J25, J28, J30, J31, J32, J33: moved to F.Cu
- J26, J27, J34: footprint Connector_PinHeader_1.00mm:PinHeader_1x01_P1.00mm_Vertical -> Connector_PinHeader_2.54mm:PinHeader_1x01_P2.54mm_Vertical; moved to F.Cu
- J7: moved to B.Cu
- J801: renamed from J4; moved to B.Cu
- J802: renamed from J8; moved to B.Cu
- Jlin1: renamed from J5; footprint Connector_PinSocket_2.00mm:PinSocket_1x01_P2.00mm_Vertical -> Connector_PinHeader_2.54mm:PinHeader_1x01_P2.54mm_Vertical
- moved D13 395.9 mm to (31.3, 69.2)
- moved D14 395.9 mm to (31.3, 73.8)
- moved D17 395.9 mm to (27.8, 69.2)
- moved D18 395.9 mm to (27.8, 73.8)
- moved RN1 395.9 mm to (29.3, 78.1)
- moved J35 386.7 mm to (29.9, 61.0)
- moved J36 386.7 mm to (29.9, 61.0)
- moved J37 386.7 mm to (29.9, 61.0)
- moved J25 360.6 mm to (38.1, 81.3), turned to 180 degrees
- moved D30 352.1 mm to (29.8, 104.1), turned to 90 degrees
- moved Jlin1 340.9 mm to (38.1, 71.1), turned to 180 degrees
- moved J26 331.2 mm to (32.4, 85.1), turned to 180 degrees
- moved J24 330.5 mm to (45.7, 48.9)
- moved J34 325.4 mm to (38.1, 86.4), turned to 180 degrees
- moved J27 323.0 mm to (38.1, 88.9), turned to 180 degrees
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- renumbered J6 to J51, J9 to JA1, J18 to JA10, J19 to JA11, J10 to JA2, J11 to JA3, J12 to JA4, J13 to JA5, J14 to JA6, J15 to JA7, J16 to JA8, J17 to JA9
Connections:
- net /2A renamed /INJ1
- net /2G renamed /INJ3
- net /2J renamed /INJ4
- net /2Q renamed /IDLE
- net /3F renamed /COIL1
- net /3I renamed /COIL2
- net /3U renamed /O2-1Heat
- net /4AH renamed /GND_SENS
- net /4R renamed /VVT
- net /AT4_UNUSED renamed /AT4
- net /LowSide1/OUT2 renamed /O2-2Heat
- net /LowSide2/OUT1 renamed /INJ5
- net /UNSUED_HALL_REF_2.5V renamed /CRANK-
- C4 pad 1: /LowSide2/OUT2 -> /INJ6
- D12 pad 1: /LowSide2/OUT2 -> /INJ6
- D6 pad 2: /LowSide2/OUT2 -> /INJ6
- J2 pad 1: /LowSide2/OUT2 -> /TACH
- P1 pad 1: (no net) -> Net-(P1-Pad1)
- P1 pad 10: (no net) -> Net-(P1-Pad10)
- P1 pad 11: (no net) -> Net-(P1-Pad11)
- P1 pad 12: (no net) -> Net-(P1-Pad12)
- P1 pad 13: (no net) -> Net-(P1-Pad13)
- P1 pad 14: (no net) -> Net-(P1-Pad14)
- P1 pad 15: (no net) -> Net-(P1-Pad15)
- P1 pad 16: (no net) -> Net-(P1-Pad16)
- P1 pad 17: (no net) -> Net-(P1-Pad17)
- P1 pad 18: (no net) -> Net-(P1-Pad18)
- P1 pad 19: (no net) -> Net-(P1-Pad19)
- P1 pad 2: (no net) -> Net-(P1-Pad2)
- P1 pad 20: (no net) -> Net-(P1-Pad20)
- P1 pad 21: (no net) -> Net-(P1-Pad21)
- P1 pad 22: (no net) -> Net-(P1-Pad22)
- P1 pad 23: (no net) -> Net-(P1-Pad23)
- P1 pad 24: (no net) -> Net-(P1-Pad24)
- P1 pad 25: (no net) -> Net-(P1-Pad25)
- P1 pad 26: (no net) -> Net-(P1-Pad26)
- P1 pad 27: (no net) -> Net-(P1-Pad27)
- P1 pad 28: (no net) -> Net-(P1-Pad28)
- P1 pad 29: (no net) -> Net-(P1-Pad29)
- P1 pad 3: (no net) -> Net-(P1-Pad3)
- P1 pad 30: (no net) -> Net-(P1-Pad30)
- P1 pad 31: (no net) -> Net-(P1-Pad31)
- P1 pad 32: (no net) -> Net-(P1-Pad32)
- P1 pad 33: (no net) -> Net-(P1-Pad33)
- P1 pad 34: (no net) -> Net-(P1-Pad34)
- P1 pad 35: (no net) -> Net-(P1-Pad35)
- P1 pad 36: (no net) -> Net-(P1-Pad36)
- P1 pad 37: (no net) -> Net-(P1-Pad37)
- P1 pad 38: (no net) -> Net-(P1-Pad38)
- P1 pad 39: (no net) -> Net-(P1-Pad39)
- P1 pad 4: (no net) -> Net-(P1-Pad4)
- P1 pad 40: (no net) -> Net-(P1-Pad40)
- P1 pad 41: (no net) -> Net-(P1-Pad41)
- P1 pad 42: (no net) -> Net-(P1-Pad42)
- P1 pad 43: (no net) -> Net-(P1-Pad43)
- P1 pad 44: (no net) -> Net-(P1-Pad44)
- P1 pad 45: (no net) -> Net-(P1-Pad45)
- P1 pad 46: (no net) -> Net-(P1-Pad46)
- P1 pad 47: (no net) -> Net-(P1-Pad47)
- P1 pad 48: (no net) -> Net-(P1-Pad48)
- P1 pad 49: (no net) -> Net-(P1-Pad49)
- P1 pad 5: (no net) -> Net-(P1-Pad5)
- P1 pad 50: (no net) -> Net-(P1-Pad50)
- P1 pad 51: (no net) -> Net-(P1-Pad51)
- P1 pad 52: (no net) -> Net-(P1-Pad52)
- P1 pad 53: (no net) -> Net-(P1-Pad53)
- P1 pad 54: (no net) -> Net-(P1-Pad54)
- P1 pad 55: (no net) -> Net-(P1-Pad55)
- P1 pad 56: (no net) -> Net-(P1-Pad56)
- P1 pad 57: (no net) -> Net-(P1-Pad57)
- P1 pad 58: (no net) -> Net-(P1-Pad58)
- P1 pad 59: (no net) -> Net-(P1-Pad59)
- P1 pad 6: (no net) -> Net-(P1-Pad6)
- P1 pad 60: (no net) -> Net-(P1-Pad60)
- P1 pad 61: (no net) -> Net-(P1-Pad61)
- P1 pad 62: (no net) -> Net-(P1-Pad62)
- P1 pad 63: (no net) -> Net-(P1-Pad63)
- P1 pad 64: (no net) -> Net-(P1-Pad64)
- P1 pad 65: (no net) -> Net-(P1-Pad65)
- P1 pad 66: (no net) -> Net-(P1-Pad66)
- P1 pad 67: (no net) -> Net-(P1-Pad67)
- P1 pad 68: (no net) -> Net-(P1-Pad68)
- P1 pad 7: (no net) -> Net-(P1-Pad7)
- P1 pad 8: (no net) -> Net-(P1-Pad8)
- P1 pad 9: (no net) -> Net-(P1-Pad9)
- U2 pad 6: /LowSide2/OUT2 -> /INJ6
- U3 pad 13: /3M -> /ALTERNATOR
- U3 pad 14: /3O -> /TACH
- U3 pad 15: /3W -> /USBD-
- U3 pad 16: /3X -> /USBD+
- U3 pad 18: /4P -> /CLT
- U3 pad 23: /4N -> /IAT
- U3 pad 25: /3V -> /CAM
- U3 pad 26: /4V -> /TPS
- U3 pad 27: /4U -> /MAP
- U3 pad 29: /3H -> /MAIN_RELAY_CONTROL
- U3 pad 32: /2O -> /AFR
- U3 pad 33: /2R -> /MIL
- U3 pad 34: /2B -> /FAN
- U3 pad 35: /2M -> /FUEL_RELAY
- U3 pad 38: /2D -> /INJ2
- U3 pad 39: /4K -> /5V_SENS2
- U3 pad 43: /2C -> /AC_FAN
- U3 pad 44: /4L -> /5V_SENS1
- U3 pad 45: /3Y -> /CRANK+
- U3 pad 47: /3N -> /CAN_L
- U3 pad 48: /3L -> /CAN_H
- U3 pad J10: (no net) -> Net-(J10-Pad1)
- U3 pad J11: (no net) -> Net-(J11-Pad1)
- U3 pad J14: (no net) -> Net-(J14-Pad1)
- U3 pad J16: (no net) -> Net-(J16-Pad1)
- U3 pad J18: (no net) -> Net-(J18-Pad1)
- U3 pad J201: (no net) -> /J201
- U3 pad J202: (no net) -> /J202
- U3 pad J203: (no net) -> /J203
- U3 pad J204: (no net) -> /J204
- U3 pad J205: (no net) -> /J205
- U3 pad J206: (no net) -> /J206
- U3 pad J207: (no net) -> /J207
- U3 pad J208: (no net) -> /J208
- U3 pad J209: (no net) -> /J209
- U3 pad J210: (no net) -> /J210
- U3 pad J6: (no net) -> Net-(J6-Pad1)
- U3 pad J9: (no net) -> Net-(J9-Pad1)
Routing:
- net +12V: track 337.6 -> 99.7 mm, vias 1 -> 0
- net /COIL2: track 150.2 -> 0.00 mm
- net Net-(W3C1-Pad1): track 111.3 -> 0.00 mm
- net /2R: track 105.2 -> 0.00 mm
- net /2C: track 104.8 -> 0.00 mm
- net /INJ4: track 98.6 -> 0.00 mm, vias 1 -> 0
- net /COIL1: track 94.6 -> 0.00 mm, vias 2 -> 0
- net /4N: track 93.2 -> 0.00 mm
- net /2O: track 91.8 -> 0.00 mm
- net /GND_SENS: track 91.2 -> 0.00 mm, vias 2 -> 0
- net /3W: track 90.9 -> 0.00 mm, vias 1 -> 0
- net /J807_PA15: track 88.1 -> 0.00 mm, vias 2 -> 0
- net Net-(W3F1-Pad1): track 86.6 -> 0.00 mm, vias 1 -> 0
- net /O2-1Heat: track 84.8 -> 0.00 mm, vias 1 -> 0
- net /4K: track 81.2 -> 0.00 mm
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Other:
- net class 12v added: clearance 0.3048, trace_width 0.59944, via_dia 0.6, via_drill 0.3
- net class 1A EXTERNAL 1oz removed
- net class 1A_EXTERNAL_1oz added: clearance 0.3048, trace_width 0.3048, via_dia 0.6858, via_drill 0.3302
- net class 2.5A EXTERNAL removed
- net class 3,5A EXT HIGH VOLTAGE removed
- net class 3.5A EXTERNAL 1oz removed
- net class 5A EXTERNAL 1oz removed
- net class CUSTOM removed
- net class CUSTOM 0.6 removed
- net class Default: clearance 0.1524 -> 0.3048
- net class INJ added: clearance 0.3048, trace_width 0.59944, via_dia 1, via_drill 0.4
- net class MIN_EXTERN_188A removed
- net class MIN_EXTERN_241A removed
- rule trace_clearance: 0.1524 -> 0.3048
- board text added: "10"
- board text added: "2"
- board text added: "20"
- board text added: "23"
- board text added: "24"
- board text added: "30"
- board text added: "40"
- board text added: "45"
- board text added: "46"
- board text added: "50"
- board text added: "5VS1"
- board text added: "60"
- board text added: "68"
- board text added: "ACFAN"
- board text added: "AFR"
- board text added: "AV10"
- board text added: "AV3"
- board text added: "AV7"
- board text added: "CANH"
- board text added: "CANL"
- board text added: "COIL1"
- board text added: "COIL2"
- board text added: "CRNK+"
- board text added: "FAN"
- board text added: "GNDS"
- board text added: "MAP"
- board text added: "USB+"
- board text added: "USB-"
- board text added: "VVT"
- board text added: "W1"
- board text added: "W10"
- board text added: "W11"
- board text added: "W12"
- board text added: "W13"
- board text added: "W14"
- board text added: "W15"
- board text added: "W16"
- board text added: "W17"
- board text added: "W18"
- board text added: "W19"
- board text added: "W2"
- board text added: "W20"
- board text added: "W21"
- board text added: "W22"
- board text added: "W23"
- board text added: "W24"
- board text added: "W25"
- board text added: "W26"
- board text added: "W27"
- board text added: "W28"
- board text added: "W29"
- board text added: "W3"
- board text added: "W30"
- board text added: "W31"
- board text added: "W32"
- board text added: "W33"
- board text added: "W34"
- board text added: "W35"
- board text added: "W36"
- board text added: "W37"
- board text added: "W38"
- board text added: "W39"
- board text added: "W4"
- board text added: "W40"
- board text added: "W41"
- board text added: "W42"
- board text added: "W43"
- board text added: "W44"
- board text added: "W45"
- board text added: "W46"
- board text added: "W47"
- board text added: "W48"
- board text added: "W49"
- board text added: "W5"
- board text added: "W50"
- board text added: "W51"
- board text added: "W52"
- board text added: "W53"
- board text added: "W54"
- board text added: "W55"
- board text added: "W56"
- board text added: "W57"
- board text added: "W58"
- board text added: "W59"
- board text added: "W6"
- board text added: "W60"
- board text added: "W61"
- board text added: "W62"
- board text added: "W63"
- board text added: "W64"
- board text added: "W65"
- board text added: "W66"
- board text added: "W67"
- board text added: "W68"
- board text added: "W7"
- board text added: "W8"
- board text added: "W9"
- board text removed: "2A"
- board text removed: "2B"
- board text removed: "2C"
- board text removed: "2D"
- board text removed: "2E"
- board text removed: "2F"
- board text removed: "2G"
- board text removed: "2H"
- board text removed: "2I"
- board text removed: "2J"
- board text removed: "2K"
- board text removed: "2M"
- board text removed: "2N"
- board text removed: "2O"
- board text removed: "2P"
- board text removed: "2Q"
- board text removed: "2R"
- board text removed: "3A"
- board text removed: "3B"
- board text removed: "3C"
- board text removed: "3D"
- board text removed: "3E"
- board text removed: "3F"
- board text removed: "3H"
- board text removed: "3I"
- board text removed: "3J"
- board text removed: "3K"
- board text removed: "3L"
- board text removed: "3M"
- board text removed: "3N"
- board text removed: "3O"
- board text removed: "3P"
- board text removed: "3Q"
- board text removed: "3S"
- board text removed: "3T"
- board text removed: "3U"
- board text removed: "3V"
- board text removed: "3W"
- board text removed: "3X"
- board text removed: "3Y"
- board text removed: "3Z"
- board text removed: "4A"
- board text removed: "4AA"
- board text removed: "4AB"
- board text removed: "4AC"
- board text removed: "4AD"
- board text removed: "4AE"
- board text removed: "4AF"
- board text removed: "4AG"
- board text removed: "4AH"
- board text removed: "4B"
- board text removed: "4C"
- board text removed: "4D"
- board text removed: "4E"
- board text removed: "4F"
- board text removed: "4H"
- board text removed: "4I"
- board text removed: "4J"
- board text removed: "4K"
- board text removed: "4L"
- board text removed: "4M"
- board text removed: "4N"
- board text removed: "4O"
- board text removed: "4P"
- board text removed: "4R"
- board text removed: "4S"
- board text removed: "4T"
- board text removed: "4U"
- board text removed: "4V"
- board text removed: "4W"
- board text removed: "4X"
- board text removed: "4Z"
- board text removed: "GP3"
- board text removed: "HALL REF 2.5V"

Commit message: R0.1 draft, pre-auto-route
Parts:
- moved J67 2.54 mm to (38.1, 73.7)
- moved J68 2.54 mm to (38.1, 76.2)
Routing:
- net +12V: track 99.7 -> 348.9 mm, vias 0 -> 4
- net GND: track 0.00 -> 221.2 mm, vias 0 -> 12
- net /COIL2: track 0.00 -> 60.4 mm
- net /VVT: track 0.00 -> 33.4 mm
- net Net-(Jlin1-Pad1): track 0.00 -> 25.6 mm
- net /AV5_UNUSED: track 0.00 -> 23.3 mm
- net /AFR: track 0.00 -> 23.3 mm
- net /GND_SENS: track 0.00 -> 21.5 mm
- net /MAP: track 0.00 -> 20.8 mm
- net /5V_SENS2: track 0.00 -> 20.8 mm
- net /ETB1: track 0.00 -> 18.4 mm
- net /AV7_UNUSED: track 0.00 -> 18.2 mm
- net /CAN_H: track 0.00 -> 18.1 mm
- net /AT3_UNUSED: track 0.00 -> 18.0 mm
- net /AV9_UNUSED: track 0.00 -> 18.0 mm
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Other:
- net class 12v: clearance 0.3048 -> 0.2032
- net class 1A_EXTERNAL_1oz: clearance 0.3048 -> 0.2032
- net class Default: clearance 0.3048 -> 0.2032
- net class INJ: clearance 0.3048 -> 0.2032; trace_width 0.59944 -> 0.6096
- rule trace_clearance: 0.3048 -> 0.2032
- board text added: "IDLE"

Commit message: R0.1 draft, pre-auto-route
Parts:
- moved J30 28.0 mm to (60.3, 94.0), turned to 0 degrees
Routing:
- net /AV5_UNUSED: track 23.3 -> 0.00 mm
Other:
- net class 12v: clearance 0.2032 -> 0.1778
- net class 1A_EXTERNAL_1oz: clearance 0.2032 -> 0.1778
- net class Default: clearance 0.2032 -> 0.1778
- net class INJ: clearance 0.2032 -> 0.1778; trace_width 0.6096 -> 0.5334
- rule trace_clearance: 0.2032 -> 0.1778
Changed lines of the file:
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@@
     (thickness 1.6)
     (drawings 215)
-    (tracks 311)
+    (tracks 306)
     (zones 0)
     (modules 201)
@@
   )
   (setup
-    (last_trace_width 0.6096)
+    (last_trace_width 0.2032)
     (user_trace_width 0.2032)
     (user_trace_width 0.2159)
@@
     (user_trace_width 2.54)
     (user_trace_width 2.7178)
-    (trace_clearance 0.2032)
+    (trace_clearance 0.1778)
     (zone_clearance 0.1524)
     (zone_45_only no)
@@
   (net 218 "Net-(Jlin1-Pad1)")
   (net_class Default "This is the default net class."
-    (clearance 0.2032)
+    (clearance 0.1778)
     (trace_width 0.2032)
     (via_dia 0.6)
@@
   )
   (net_class 12v ""
-    (clearance 0.2032)
+    (clearance 0.1778)
     (trace_width 0.59944)
     (via_dia 0.6)
@@
   )
   (net_class 1A_EXTERNAL_1oz ""
-    (clearance 0.2032)
+    (clearance 0.1778)
     (trace_width 0.3048)
     (via_dia 0.6858)
@@
     (add_net "Net-(J7-Pad5)")
     (add_net "Net-(J9-Pad1)")
-    (add_net "Net-(JA3-Pad1)")
-    (add_net "Net-(JA3-Pad3)")
-    (add_net "Net-(JA3-Pad5)")
-    (add_net "Net-(JA3-Pad7)")
     (add_net "Net-(Jlin1-Pad1)")
     (add_net "Net-(P1-Pad1)")
@@
   )
   (net_class INJ ""
-    (clearance 0.2032)
-    (trace_width 0.6096)
+    (clearance 0.1778)
+    (trace_width 0.5334)
     (via_dia 1)
     (via_drill 0.4)
@@
   )
   (module Connector_PinHeader_2.54mm:PinHeader_1x01_P2.54mm_Vertical (layer F.Cu)
-    (at 32.385 95.25 180)
+    (at 60.325 93.98)
     (descr "Through hole straight pin header, 1x01, 2.54mm pitch, single row")
     (tags "Through hole pin header THT 1x01 2.54mm single row")
@@
     (fp_line (start 1.27 -1.27) (end 1.27 1.27) (layer F.Fab) (width 0.1))
     (fp_line (start -0.635 -1.27) (end 1.27 -1.27) (layer F.Fab) (width 0.1))
-    (pad 1 thru_hole rect (at 0 0 180) (size 1.7 1.7) (drill 1) (layers *.Cu *.Mask)
+    (pad 1 thru_hole rect (at 0 0) (size 1.7 1.7) (drill 1) (layers *.Cu *.Mask)
       (net 55 /AV5_UNUSED))
     (model ${KISYS3DMOD}/Connector_PinHeader_2.54mm.3dshapes/PinHeader_1x01_P2.54mm_Vertical.wrl
@@
     (effects (font (size 0.75 0.75) (thickness 0.13)) (justify mirror))
   )
-  (gr_text AV5 (at 29.845 94.615) (layer B.SilkS)
+  (gr_text AV5 (at 62.865 94.615 180) (layer B.SilkS)
     (effects (font (size 0.75 0.75) (thickness 0.15)) (justify mirror))
   )
@@
     (effects (font (size 0.75 0.75) (thickness 0.13)))
   )
-  (gr_text AV5 (at 29.845 94.615) (layer F.SilkS)
+  (gr_text AV5 (at 62.865 94.615 180) (layer F.SilkS)
     (effects (font (size 0.75 0.75) (thickness 0.15)))
   )
@@
   (segment (start 90.805 45.085) (end 90.805 40.64) (width 0.6096) (layer B.Cu) (net 1))
   (segment (start 92.075 46.355) (end 90.805 45.085) (width 0.6096) (layer B.Cu) (net 1))
-  (segment (start 31.322 72.9945) (end 31.322 70.66) (width 0.6) (layer F.Cu) (net 33))
-  (segment (start 27.766 72.9945) (end 27.766 70.66) (width 0.6) (layer F.Cu) (net 35))
-  (segment (start 30.494801 74.921699) (end 30.494801 77.2) (width 0.6) (layer F.Cu) (net 43))
-  (segment (start 31.322 74.5695) (end 30.847 74.5695) (width 0.6) (layer F.Cu) (net 43))
-  (segment (start 30.847 74.5695) (end 30.494801 74.921699) (width 0.6) (layer F.Cu) (net 43))
-  (segment (start 27.766 76.880801) (end 28.085199 77.2) (width 0.6) (layer F.Cu) (net 45))
-  (segment (start 27.766 74.5695) (end 27.766 76.880801) (width 0.6) (layer F.Cu) (net 45))
-  (segment (start 36.83 31.67) (end 38.5 30) (width 0.6) (layer B.Cu) (net 113))
-  (segment (start 36.83 36.83) (end 36.83 31.67) (width 0.6) (layer B.Cu) (net 113))
-  (segment (start 95.885 34.265) (end 96.85 33.3) (width 1.524) (layer B.Cu) (net 143))
-  (segment (start 95.885 36.83) (end 95.885 34.265) (width 1.524) (layer B.Cu) (net 143))
-  (segment (start 80.645 33.505) (end 80.85 33.3) (width 2.7178) (layer F.Cu) (net 147))
-  (segment (start 80.645 37.465) (end 80.645 33.505) (width 2.7178) (layer F.Cu) (net 147))
-  (segment (start 80.645 33.505) (end 80.85 33.3) (width 2.7178) (layer B.Cu) (net 147))
-  (segment (start 80.645 36.83) (end 80.645 33.505) (width 2.7178) (layer B.Cu) (net 147))
   (segment (start 96.443801 41.198801) (end 95.885 40.64) (width 1.524) (layer B.Cu) (net 2))
   (segment (start 47.6276 109.2226) (end 48.26 109.855) (width 1.524) (layer B.Cu) (net 2))
@@
   (segment (start 153.866 51.7085) (end 153.665 51.5075) (width 0.3048) (layer F.Cu) (net 28))
   (segment (start 153.866 53.514) (end 153.866 51.7085) (width 0.3048) (layer F.Cu) (net 28))
+  (segment (start 31.322 72.9945) (end 31.322 70.66) (width 0.6) (layer F.Cu) (net 33))
+  (segment (start 27.766 72.9945) (end 27.766 70.66) (width 0.6) (layer F.Cu) (net 35))
+  (segment (start 30.494801 74.921699) (end 30.494801 77.2) (width 0.6) (layer F.Cu) (net 43))
+  (segment (start 31.322 74.5695) (end 30.847 74.5695) (width 0.6) (layer F.Cu) (net 43))
+  (segment (start 30.847 74.5695) (end 30.494801 74.921699) (width 0.6) (layer F.Cu) (net 43))
+  (segment (start 27.766 76.880801) (end 28.085199 77.2) (width 0.6) (layer F.Cu) (net 45))
+  (segment (start 27.766 74.5695) (end 27.766 76.880801) (width 0.6) (layer F.Cu) (net 45))
   (segment (start 53.921199 80.099399) (end 54.327601 80.505801) (width 0.3048) (layer B.Cu) (net 52))
   (segment (start 40.435401 80.099399) (end 53.921199 80.099399) (width 0.3048) (layer B.Cu) (net 52))
@@
   (segment (start 53.921199 90.012201) (end 54.327601 89.605799) (width 0.3048) (layer B.Cu) (net 54))
   (segment (start 38.1 88.9) (end 39.2548 88.9) (width 0.3048) (layer B.Cu) (net 54))
-  (segment (start 54.327601 94.605799) (end 55.1276 93.8058) (width 0.3048) (layer F.Cu) (net 55))
-  (segment (start 53.921199 95.012201) (end 54.327601 94.605799) (width 0.3048) (layer F.Cu) (net 55))
-  (segment (start 47.135725 95.012201) (end 53.921199 95.012201) (width 0.3048) (layer F.Cu) (net 55))
-  (segment (start 46.897926 95.25) (end 47.135725 95.012201) (width 0.3048) (layer F.Cu) (net 55))
-  (segment (start 32.385 95.25) (end 46.897926 95.25) (width 0.3048) (layer F.Cu) (net 55))
   (segment (start 51.827601 94.605799) (end 52.6276 93.8058) (width 0.3048) (layer B.Cu) (net 56))
   (segment (start 51.421199 95.012201) (end 51.827601 94.605799) (width 0.3048) (layer B.Cu) (net 56))
@@
   (segment (start 52.4818 73.66) (end 55.1276 76.3058) (width 0.3048) (layer B.Cu) (net 90))
   (segment (start 38.1 73.66) (end 52.4818 73.66) (width 0.3048) (layer B.Cu) (net 90))
+  (segment (start 36.83 31.67) (end 38.5 30) (width 0.6) (layer B.Cu) (net 113))
+  (segment (start 36.83 36.83) (end 36.83 31.67) (width 0.6) (layer B.Cu) (net 113))
+  (segment (start 95.885 34.265) (end 96.85 33.3) (width 1.524) (layer B.Cu) (net 143))
+  (segment (start 95.885 36.83) (end 95.885 34.265) (width 1.524) (layer B.Cu) (net 143))
+  (segment (start 80.645 33.505) (end 80.85 33.3) (width 2.7178) (layer F.Cu) (net 147))
+  (segment (start 80.645 37.465) (end 80.645 33.505) (width 2.7178) (layer F.Cu) (net 147))
+  (segment (start 80.645 33.505) (end 80.85 33.3) (width 2.7178) (layer B.Cu) (net 147))
+  (segment (start 80.645 36.83) (end 80.645 33.505) (width 2.7178) (layer B.Cu) (net 147))
   (segment (start 56.896 74.422) (end 61.2014 74.422) (width 0.3048) (layer B.Cu) (net 218))
   (segment (start 38.1 71.12) (end 53.594 71.12) (width 0.3048) (layer B.Cu) (net 218))

Commit message: R0.1 draft, pre-auto-route
Routing:
- net /INJ3: track 0.00 -> 184.1 mm
- net /IDLE: track 17.0 -> 198.4 mm
- net /J804_3.3V: track 0.00 -> 154.1 mm, vias 0 -> 2
- net /INJ4: track 0.00 -> 140.1 mm, vias 0 -> 2
- net /HI4_UNUSED: track 0.00 -> 135.9 mm, vias 0 -> 2
- net /INJ1: track 0.00 -> 130.2 mm, vias 0 -> 1
- net /HI2_UNUSED: track 0.00 -> 128.7 mm
- net /AV8_UNUSED: track 0.00 -> 124.9 mm, vias 0 -> 3
- net /MIL: track 0.00 -> 101.8 mm, vias 0 -> 2
- net /J806_PB9: track 0.00 -> 99.1 mm
- net Net-(P1-Pad35): track 0.00 -> 96.4 mm, vias 0 -> 1
- net /J801_5V: track 0.00 -> 93.2 mm
- net /INJ2: track 0.00 -> 90.7 mm
- net /ETB1: track 18.4 -> 107.8 mm, vias 0 -> 1
- net /J810_PC12: track 0.00 -> 89.3 mm
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
Commit message: R0.1 draft, pre-auto-route
Routing:
- net GND: vias 358 -> 359
Changed lines of the file:
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@@
     (thickness 1.6)
     (drawings 215)
-    (tracks 1780)
+    (tracks 1781)
     (zones 0)
     (modules 201)
@@
   )
   (gr_poly (pts (xy 27.686 35.56) (xy 27.686 48.26) (xy 20.955 48.26) (xy 20.955 35.56)) (layer F.Mask) (width 0.1))
-  (gr_text "     4" (at 63.5 175.895) (layer B.Cu)
+  (gr_text "     4" (at 23.495 26.035 270) (layer B.Cu)
     (effects (font (size 1.5 1.5) (thickness 0.3)))
   )
-  (gr_text "1     " (at 63.5 175.895) (layer F.Cu)
+  (gr_text "1     " (at 23.495 26.035 270) (layer F.Cu)
     (effects (font (size 1.5 1.5) (thickness 0.3)))
   )
@@
   (via (at 40.132 42.926) (size 0.6) (drill 0.3) (layers F.Cu B.Cu) (net 1))
   (via (at 36.703 42.926) (size 0.6) (drill 0.3) (layers F.Cu B.Cu) (net 1))
-  (via (at 43.053 43.942) (size 0.6) (drill 0.3) (layers F.Cu B.Cu) (net 1))
+  (via (at 43.307 44.45) (size 0.6) (drill 0.3) (layers F.Cu B.Cu) (net 1))
   (via (at 62.103 31.75) (size 0.6) (drill 0.3) (layers F.Cu B.Cu) (net 1))
   (via (at 77.851 35.052) (size 0.6) (drill 0.3) (layers F.Cu B.Cu) (net 1))
@@
   (via (at 95.123 98.425) (size 0.6) (drill 0.3) (layers F.Cu B.Cu) (net 1))
   (via (at 98.171 101.6) (size 0.6) (drill 0.3) (layers F.Cu B.Cu) (net 1))
-  (via (at 21.59 26.67) (size 0.6) (drill 0.3) (layers F.Cu B.Cu) (net 1))
+  (via (at 26.035 31.75) (size 0.6) (drill 0.3) (layers F.Cu B.Cu) (net 1))
   (via (at 21.59 59.69) (size 0.6) (drill 0.3) (layers F.Cu B.Cu) (net 1))
   (via (at 21.59 79.375) (size 0.6) (drill 0.3) (layers F.Cu B.Cu) (net 1))
@@
   (via (at 27.305 21.59) (size 0.6) (drill 0.3) (layers F.Cu B.Cu) (net 1))
   (via (at 59.69 20.955) (size 0.6) (drill 0.3) (layers F.Cu B.Cu) (net 1))
+  (via (at 21.336 31.75) (size 0.6) (drill 0.3) (layers F.Cu B.Cu) (net 1))
   (segment (start 47.6276 109.223) (end 48.26 109.855) (width 1.524) (layer B.Cu) (net 2))
   (segment (start 48.26 109.855) (end 58.8987 109.855) (width 1.524) (layer B.Cu) (net 2))
@@
     (polygon
       (pts
-        (xy 67.945 179.07) (xy 59.055 179.07) (xy 59.055 174.625) (xy 67.945 174.625)
+        (xy 20.32 30.48) (xy 20.32 20.32) (xy 24.765 20.32) (xy 24.765 30.48)
       )
     )
