File: 68_vag_PNP.kicad_pcb (KiCad board)
At the start: 2 copper layers, 149 x 140 mm, 201 parts, among them J10 Conn_01x01, J11 Conn_01x01, J14 Conn_01x01, J16 Conn_01x01, J18 Conn_01x01, J2 Conn_01x01, J201 Conn_01x05, J202 Conn_01x05, J24 Conn_01x01, J25 Conn_01x01, J26 Conn_01x01, J27 Conn_01x01, J28 Conn_01x01, J29 Conn_01x01, J30 Conn_01x01, J31 Conn_01x01, J32 Conn_01x01, J33 Conn_01x01, J34 Conn_01x01, J35 Conn_01x01, J36 Conn_01x01, J37 Conn_01x01, J38 Conn_01x01, J39 Conn_01x01, J40 Conn_01x01, J41 Conn_01x01, J42 Conn_01x01, J45 Conn_01x01, J46 Conn_01x01, J47 Conn_01x01, J48 Conn_01x01, J49 Conn_01x01, J51 Conn_01x05, J52 Conn_01x01, J53 Conn_01x01, J56 Conn_01x01, J57 Conn_01x01, J58 Conn_01x01, J6 Conn_01x01, J62 Conn_01x01, J63 Conn_01x01, J64 Conn_01x01, J65 Conn_01x01, J67 Conn_01x01, J68 Conn_01x01, J69 Conn_01x01, J7 Conn_01x05, J70 Conn_01x01, J71 Conn_01x01, J72 Conn_01x01, J801 Conn_01x05, J802 Conn_01x05, J9 Conn_01x01, P1 1123038-2, U1 VNLD5090, U2 VNLD5090, U3 molex_48pin_MRE, U4 ITEAD_HC-05

Commit message: Updated the dimentions on the CmtsUser layer.
Other:
- board text removed: "154mm"
- board text removed: "159mm"
Changed lines of the file:
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@@
     )
+  )
+  (dimension 140 (width 0.15) (layer Cmts.User)
+    (gr_text "140.000 mm" (at 191.546 90 90) (layer Cmts.User)
+      (effects (font (size 1 1) (thickness 0.15)))
+    )
+    (feature1 (pts (xy 164 20) (xy 190.832421 20)))
+    (feature2 (pts (xy 164 160) (xy 190.832421 160)))
+    (crossbar (pts (xy 190.246 160) (xy 190.246 20)))
+    (arrow1a (pts (xy 190.246 20) (xy 190.832421 21.126504)))
+    (arrow1b (pts (xy 190.246 20) (xy 189.659579 21.126504)))
+    (arrow2a (pts (xy 190.246 160) (xy 190.832421 158.873496)))
+    (arrow2b (pts (xy 190.246 160) (xy 189.659579 158.873496)))
+  )
+  (dimension 149 (width 0.15) (layer Cmts.User)
+    (gr_text "149.000 mm" (at 94.5 170.971999) (layer Cmts.User)
+      (effects (font (size 1 1) (thickness 0.15)))
+    )
+    (feature1 (pts (xy 169 155) (xy 169 170.25842)))
+    (feature2 (pts (xy 20 155) (xy 20 170.25842)))
+    (crossbar (pts (xy 20 169.671999) (xy 169 169.671999)))
+    (arrow1a (pts (xy 169 169.671999) (xy 167.873496 170.25842)))
+    (arrow1b (pts (xy 169 169.671999) (xy 167.873496 169.085578)))
+    (arrow2a (pts (xy 20 169.671999) (xy 21.126504 170.25842)))
+    (arrow2b (pts (xy 20 169.671999) (xy 21.126504 169.085578)))
   )
   (gr_text VVT (at 24.13 100.33) (layer B.SilkS)
@@
     (effects (font (size 0.75 0.75) (thickness 0.13)))
   )
-  (gr_text 159mm (at 191.8 98.6 90) (layer Cmts.User)
-    (effects (font (size 1 1) (thickness 0.15)))
-  )
-  (gr_text 154mm (at 97.3 185) (layer Cmts.User)
-    (effects (font (size 1 1) (thickness 0.15)))
-  )
   (gr_text "FIRE EXTINGUISHER REQUIRED" (at 135.89 61.595 90) (layer F.SilkS)
     (effects (font (size 2.286 2.286) (thickness 0.2032)))
   )
-  (dimension 154.051052 (width 0.15) (layer Cmts.User)
-    (gr_text "6.0650 in" (at 97.851272 183.105839 359.9527652) (layer Cmts.User)
-      (effects (font (size 1 1) (thickness 0.15)))
-    )
-    (feature1 (pts (xy 174.879 180.467) (xy 174.87736 182.455759)))
-    (feature2 (pts (xy 20.828 180.34) (xy 20.82636 182.328759)))
-    (crossbar (pts (xy 20.826844 181.742339) (xy 174.877844 181.869339)))
-    (arrow1a (pts (xy 174.877844 181.869339) (xy 173.750857 182.454831)))
-    (arrow1b (pts (xy 174.877844 181.869339) (xy 173.751824 181.28199)))
-    (arrow2a (pts (xy 20.826844 181.742339) (xy 21.952864 182.329688)))
-    (arrow2b (pts (xy 20.826844 181.742339) (xy 21.953831 181.156847)))
-  )
-  (dimension 158.877 (width 0.15) (layer Cmts.User)
-    (gr_text "6.2550 in" (at 189.641 98.3615 90) (layer Cmts.User)
-      (effects (font (size 1 1) (thickness 0.15)))
-    )
-    (feature1 (pts (xy 177.8 18.923) (xy 188.927421 18.923)))
-    (feature2 (pts (xy 177.8 177.8) (xy 188.927421 177.8)))
-    (crossbar (pts (xy 188.341 177.8) (xy 188.341 18.923)))
-    (arrow1a (pts (xy 188.341 18.923) (xy 188.927421 20.049504)))
-    (arrow1b (pts (xy 188.341 18.923) (xy 187.754579 20.049504)))
-    (arrow2a (pts (xy 188.341 177.8) (xy 188.927421 176.673496)))
-    (arrow2b (pts (xy 188.341 177.8) (xy 187.754579 176.673496)))
+  (dimension 149 (width 0.15) (layer Cmts.User)
+    (gr_text "5.8661 in" (at 94.5 168.559) (layer Cmts.User)
+      (effects (font (size 1 1) (thickness 0.15)))
+    )
+    (feature1 (pts (xy 169 155) (xy 169 167.845421)))
+    (feature2 (pts (xy 20 155) (xy 20 167.845421)))
+    (crossbar (pts (xy 20 167.259) (xy 169 167.259)))
+    (arrow1a (pts (xy 169 167.259) (xy 167.873496 167.845421)))
+    (arrow1b (pts (xy 169 167.259) (xy 167.873496 166.672579)))
+    (arrow2a (pts (xy 20 167.259) (xy 21.126504 167.845421)))
+    (arrow2b (pts (xy 20 167.259) (xy 21.126504 166.672579)))
+  )
+  (dimension 140 (width 0.15) (layer Cmts.User)
+    (gr_text "5.5118 in" (at 188.752 90 90) (layer Cmts.User)
+      (effects (font (size 1 1) (thickness 0.15)))
+    )
+    (feature1 (pts (xy 164 20) (xy 188.038421 20)))
+    (feature2 (pts (xy 164 160) (xy 188.038421 160)))
+    (crossbar (pts (xy 187.452 160) (xy 187.452 20)))
+    (arrow1a (pts (xy 187.452 20) (xy 188.038421 21.126504)))
+    (arrow1b (pts (xy 187.452 20) (xy 186.865579 21.126504)))
+    (arrow2a (pts (xy 187.452 160) (xy 188.038421 158.873496)))
+    (arrow2b (pts (xy 187.452 160) (xy 186.865579 158.873496)))
   )
   (gr_text "microRusEfi 68 Vag PnP 0.1" (at 22.225 69.215 90) (layer F.SilkS)
